File: communication.kicad_sch (KiCad schematic)
At the start: 16 parts, among them X1 ASCO

Commit message: 1YN BT/WLAN connections
Connections:
- net BT_PCM_SDO: now reaches U1.10 (BT_PCM_OUT)
- net BT_PCM_CLK: now reaches U1.11 (BT_PCM_CLK)
- net BT_REG_ON: now reaches U1.14 (BT_REG_ON)
- net WL_HOST_WAKE: now reaches U1.27 (WL_GPIO_0_HOST_WAKE)
- net WL_REG_ON: now reaches U1.28 (WL_REG_ON)
- net BT_HOST_WAKE: now reaches U1.38 (BT_HOST_WAKE)
- net BT_DEV_WAKE: now reaches U1.39 (BT_DEV_WAKE)
- net BT_PCM_WS: now reaches U1.8 (BT_PCM_SYNC)
- net BT_PCM_SDI: now reaches U1.9 (BT_PCM_IN)
- no-connect marks 0 -> 2
Changed lines of the file:
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@@
   (junction (at 143.51 123.19) (diameter 0) (color 0 0 0 0)
   )
+  (no_connect (at 77.47 132.08))
+  (no_connect (at 77.47 134.62))
   (wire (pts (xy 88.9 22.86) (xy 95.25 22.86))
     (stroke (width 0) (type default))
@@
     (stroke (width 0) (type default))
   )
+  (wire (pts (xy 77.47 114.3) (xy 80.01 114.3))
+    (stroke (width 0) (type default))
+  )
   (wire (pts (xy 143.51 72.39) (xy 143.51 73.66))
     (stroke (width 0) (type default))
@@
     (stroke (width 0) (type dash))
   )
+  (wire (pts (xy 77.47 139.7) (xy 80.01 139.7))
+    (stroke (width 0) (type default))
+  )
   (wire (pts (xy 77.47 154.94) (xy 80.01 154.94))
     (stroke (width 0) (type default))
@@
     (stroke (width 0) (type default))
   )
+  (wire (pts (xy 77.47 119.38) (xy 80.01 119.38))
+    (stroke (width 0) (type default))
+  )
   (wire (pts (xy 129.54 30.48) (xy 130.81 30.48))
     (stroke (width 0) (type default))
@@
     (stroke (width 0) (type dash))
   )
+  (wire (pts (xy 77.47 111.76) (xy 80.01 111.76))
+    (stroke (width 0) (type default))
+  )
   (polyline (pts (xy 50.8 50.8) (xy 50.8 12.7))
     (stroke (width 0) (type dash))
@@
     (stroke (width 0) (type default))
   )
+  (wire (pts (xy 77.47 121.92) (xy 80.01 121.92))
+    (stroke (width 0) (type default))
+  )
   (wire (pts (xy 76.2 31.75) (xy 76.2 29.21))
     (stroke (width 0) (type default))
@@
     (stroke (width 0) (type default))
   )
+  (wire (pts (xy 77.47 127) (xy 80.01 127))
+    (stroke (width 0) (type default))
+  )
   (polyline (pts (xy 114.3 50.8) (xy 165.1 50.8))
     (stroke (width 0) (type dash))
@@
     (stroke (width 0) (type dash))
   )
+  (wire (pts (xy 77.47 124.46) (xy 80.01 124.46))
+    (stroke (width 0) (type default))
+  )
   (wire (pts (xy 132.08 78.74) (xy 132.08 80.01))
     (stroke (width 0) (type default))
@@
     (stroke (width 0) (type default))
   )
+  (wire (pts (xy 77.47 116.84) (xy 80.01 116.84))
+    (stroke (width 0) (type default))
+  )
   (polyline (pts (xy 12.7 63.5) (xy 12.7 190.5))
     (stroke (width 0) (type dash))
@@
     (stroke (width 0) (type dash))
   )
+  (wire (pts (xy 77.47 137.16) (xy 80.01 137.16))
+    (stroke (width 0) (type default))
+  )
   (wire (pts (xy 88.9 22.86) (xy 88.9 24.13))
     (stroke (width 0) (type default))
@@
     )
   )
+  (global_label "BT_REG_ON" (shape input) (at 80.01 121.92 0) (fields_autoplaced)
+    (effects (font (size 1.27 1.27)) (justify left))
+    (property "Intersheetrefs" "${INTERSHEET_REFS}" (at 93.4386 121.92 0)
+      (effects (font (size 1.27 1.27)) (justify left) hide)
+    )
+  )
   (global_label "VDD_1YN" (shape input) (at 52.07 91.44 90) (fields_autoplaced)
     (effects (font (size 1.27 1.27)) (justify left))
@@
     )
   )
+  (global_label "BT_PCM_CLK" (shape input) (at 80.01 119.38 0) (fields_autoplaced)
+    (effects (font (size 1.27 1.27)) (justify left))
+    (property "Intersheetrefs" "${INTERSHEET_REFS}" (at 94.6481 119.38 0)
+      (effects (font (size 1.27 1.27)) (justify left) hide)
+    )
+  )
   (global_label "1YN_DATA0" (shape input) (at 80.01 152.4 0) (fields_autoplaced)
     (effects (font (size 1.27 1.27)) (justify left))
@@
     )
   )
+  (global_label "BT_DEV_WAKE" (shape input) (at 80.01 127 0) (fields_autoplaced)
+    (effects (font (size 1.27 1.27)) (justify left))
+    (property "Intersheetrefs" "${INTERSHEET_REFS}" (at 95.5552 127 0)
+      (effects (font (size 1.27 1.27)) (justify left) hide)
+    )
+  )
   (global_label "VDD_1YN" (shape input) (at 21.59 36.83 90) (fields_autoplaced)
     (effects (font (size 1.27 1.27)) (justify left))
@@
     )
   )
+  (global_label "WL_HOST_WAKE" (shape input) (at 80.01 137.16 0) (fields_autoplaced)
+    (effects (font (size 1.27 1.27)) (justify left))
+    (property "Intersheetrefs" "${INTERSHEET_REFS}" (at 97.1276 137.16 0)
+      (effects (font (size 1.27 1.27)) (justify left) hide)
+    )
+  )
+  (global_label "WL_REG_ON" (shape input) (at 80.01 139.7 0) (fields_autoplaced)
+    (effects (font (size 1.27 1.27)) (justify left))
+    (property "Intersheetrefs" "${INTERSHEET_REFS}" (at 93.6805 139.7 0)
+      (effects (font (size 1.27 1.27)) (justify left) hide)
+    )
+  )
+  (global_label "BT_PCM_SDO" (shape input) (at 80.01 116.84 0) (fields_autoplaced)
+    (effects (font (size 1.27 1.27)) (justify left))
+    (property "Intersheetrefs" "${INTERSHEET_REFS}" (at 94.89 116.84 0)
+      (effects (font (size 1.27 1.27)) (justify left) hide)
+    )
+  )
   (global_label "SR_VLX" (shape input) (at 129.54 149.86 180) (fields_autoplaced)
     (effects (font (size 1.27 1.27)) (justify right))
@@
     )
   )
+  (global_label "BT_HOST_WAKE" (shape input) (at 80.01 124.46 0) (fields_autoplaced)
+    (effects (font (size 1.27 1.27)) (justify left))
+    (property "Intersheetrefs" "${INTERSHEET_REFS}" (at 96.8857 124.46 0)
+      (effects (font (size 1.27 1.27)) (justify left) hide)
+    )
+  )
   (global_label "ANT" (shape input) (at 30.48 109.22 180) (fields_autoplaced)
     (effects (font (size 1.27 1.27)) (justify right))
@@
     )
   )
+  (global_label "BT_PCM_WS" (shape input) (at 80.01 111.76 0) (fields_autoplaced)
+    (effects (font (size 1.27 1.27)) (justify left))
+    (property "Intersheetrefs" "${INTERSHEET_REFS}" (at 93.7409 111.76 0)
+      (effects (font (size 1.27 1.27)) (justify left) hide)
+    )
+  )
   (global_label "GND_SR_PVSS" (shape input) (at 132.08 123.19 180) (fields_autoplaced)
     (effects (font (size 1.27 1.27)) (justify right))
@@
       (effects (font (size 1.27 1.27)) (justify left) hide)
     )
+  )
+  (global_label "BT_PCM_SDI" (shape input) (at 80.01 114.3 0) (fields_autoplaced)
+    (effects (font (size 1.27 1.27)) (justify left))
+    (property "Intersheetrefs" "${INTERSHEET_REFS}" (at 94.1643 114.3 0)
+      (effects (font (size 1.27 1.27)) (justify left) hide)
+    )
