File: BLE + NFC.kicad_sch (KiCad schematic)
At the start: 16 parts, among them IC5 nRF52832-CIAA-G-R7, Y2 Crystal_GND24

Commit message: updated BLE + NFC.kicad_sch
- added pins for I2C slave communication
- added connections to I2C pins and SWD/JTAG interface
Connections:
- net NRF_SWCLK: now reaches IC5.F1 (SWDCLK)
- net NRF_SDA: now reaches IC5.F6 (P0.07)
- net NRF_SCL: now reaches IC5.F7 (P0.06)
- net NRF_SWDIO: now reaches IC5.G1 (SWDIO)
- net NRF_NRST: now reaches IC5.H1 (P0.21_/NRESET)
Other:
- note added: "P0.22 - P0.31 do not use (only low frequency capable, ds. p. 18)"
Changed lines of the file:
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@@
+    (stroke (width 0) (type default))
+  )
+  (wire (pts (xy 115.57 96.52) (xy 120.65 96.52))
     (stroke (width 0) (type default))
   )
@@
     (stroke (width 0) (type default))
   )
+  (wire (pts (xy 176.53 118.11) (xy 179.07 118.11))
+    (stroke (width 0) (type default))
+  )
   (wire (pts (xy 102.87 111.76) (xy 105.41 111.76))
     (stroke (width 0) (type default))
@@
     (stroke (width 0) (type default))
   )
+  (wire (pts (xy 176.53 115.57) (xy 179.07 115.57))
+    (stroke (width 0) (type default))
+  )
+  (wire (pts (xy 115.57 99.06) (xy 120.65 99.06))
+    (stroke (width 0) (type default))
+  )
   (wire (pts (xy 166.37 43.18) (xy 165.1 43.18))
     (stroke (width 0) (type default))
   )
+  (wire (pts (xy 115.57 101.6) (xy 120.65 101.6))
+    (stroke (width 0) (type default))
+  )
   (wire (pts (xy 44.45 30.48) (xy 40.64 30.48))
     (stroke (width 0) (type default))
@@
     (stroke (width 0) (type default))
     (fill (type none))
+  )
+  (text "P0.22 - P0.31 do not use (only low frequency capable, ds. p. 18)"
+    (at 101.6 158.75 0)
+    (effects (font (size 1.27 1.27)) (justify left bottom))
   )
   (text "TBD:\n\n- programming interface\n- i2c slave connections"
@@
     )
   )
+  (hierarchical_label "NRF_SWCLK" (shape input) (at 115.57 99.06 180) (fields_autoplaced)
+    (effects (font (size 1.27 1.27)) (justify right))
+    (property "Intersheetrefs" "${INTERSHEET_REFS}" (at 102.541 99.06 0)
+      (effects (font (size 1.27 1.27)) (justify right) hide)
+    )
+  )
+  (hierarchical_label "NRF_SCL" (shape input) (at 179.07 118.11 0) (fields_autoplaced)
+    (effects (font (size 1.27 1.27)) (justify left))
+    (property "Intersheetrefs" "${INTERSHEET_REFS}" (at 190.1401 118.11 0)
+      (effects (font (size 1.27 1.27)) (justify left) hide)
+    )
+  )
   (hierarchical_label "NFC_ANT2" (shape input) (at 119.38 78.74 180) (fields_autoplaced)
     (effects (font (size 1.27 1.27)) (justify right))
@@
     )
   )
+  (hierarchical_label "NRF_SDA" (shape input) (at 179.07 115.57 0) (fields_autoplaced)
+    (effects (font (size 1.27 1.27)) (justify left))
+    (property "Intersheetrefs" "${INTERSHEET_REFS}" (at 190.2006 115.57 0)
+      (effects (font (size 1.27 1.27)) (justify left) hide)
+    )
+  )
   (hierarchical_label "NFC_ANT1" (shape input) (at 119.38 76.2 180) (fields_autoplaced)
     (effects (font (size 1.27 1.27)) (justify right))
@@
       (effects (font (size 1.27 1.27)) (justify right) hide)
     )
+  )
+  (hierarchical_label "NRF_SWDIO" (shape input) (at 115.57 101.6 180) (fields_autoplaced)
+    (effects (font (size 1.27 1.27)) (justify right))
+    (property "Intersheetrefs" "${INTERSHEET_REFS}" (at 102.9038 101.6 0)
+      (effects (font (size 1.27 1.27)) (justify right) hide)
+    )
+  )
+  (hierarchical_label "NRF_NRST" (shape input) (at 115.57 96.52 180) (fields_autoplaced)
+    (effects (font (size 1.27 1.27)) (justify right))
+    (property "Intersheetrefs" "${INTERSHEET_REFS}" (at 103.9924 96.52 0)
+      (effects (font (size 1.27 1.27)) (justify right) hide)
+    )

Commit message: Update JTAG
Add Footprint for JTAG connector
Add NRF connections
Connections:
- net NRF_RXD: now reaches IC5.F4 (P0.11)
- net NRF_TXD: now reaches IC5.H6 (P0.12)
Other:
- note removed: "please check footprint of antenna!"
Changed lines of the file:
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@@
+    (stroke (width 0) (type default))
+  )
+  (wire (pts (xy 176.53 107.95) (xy 179.07 107.95))
     (stroke (width 0) (type default))
   )
@@
   )
   (wire (pts (xy 154.94 43.18) (xy 154.94 45.72))
+    (stroke (width 0) (type default))
+  )
+  (wire (pts (xy 176.53 110.49) (xy 179.07 110.49))
     (stroke (width 0) (type default))
   )
@@
     (effects (font (size 1.27 1.27)) (justify left bottom))
   )
-  (text "please check footprint of antenna!" (at 52.07 44.45 0)
-    (effects (font (size 1.27 1.27) (thickness 0.254) bold (color 255 0 21 1)) (justify right bottom))
-  )
   (global_label "DEC2" (shape input) (at 157.48 43.18 90) (fields_autoplaced)
     (effects (font (size 1.27 1.27)) (justify left))
@@
     )
   )
+  (hierarchical_label "NRF_TXD" (shape input) (at 179.07 107.95 0) (fields_autoplaced)
+    (effects (font (size 1.27 1.27)) (justify left))
+    (property "Intersheetrefs" "${INTERSHEET_REFS}" (at 189.3965 107.95 0)
+      (effects (font (size 1.27 1.27)) (justify left) hide)
+    )
+  )
+  (hierarchical_label "NRF_RXD" (shape input) (at 179.07 110.49 0) (fields_autoplaced)
+    (effects (font (size 1.27 1.27)) (justify left))
+    (property "Intersheetrefs" "${INTERSHEET_REFS}" (at 189.6989 110.49 0)
+      (effects (font (size 1.27 1.27)) (justify left) hide)
+    )
+  )
