File: 9dof.kicad_sch (KiCad schematic)
At the start: 8 parts, among them IC2 BMI323, U3 BMM350

Commit message: progressed layout and made changes in bmi323 (set unconnected pins to NC) + changed debug connections in preparation to make bridges to debug part + changed VSYS, VUSB, VBAT+ and other connected power traces to 0.2mm trace thickness + added BMI323 layout + moved MAX30102 to make space for caps + added missing caps to MAX30102 + changed gpio order for better layout + added BMM350 layout next to BMI323
Parts:
- IC2: Manufacturer_Name (none) -> BOSCH; Manufacturer_Part_Number (none) -> BMI323; Mouser Part Number (none) -> 262-BMI323; Mouser Price/Stock (none) -> https://www.mouser.co.uk/ProductDetail/Bosch-Sensortec/BMI3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
- R3: footprint Resistor_SMD:R_0201_0603Metric_Pad0.64x0.40mm_HandSolder -> Resistor_SMD:R_0201_0603Metric
Changed lines of the file:
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@@
       (effects (font (size 1.27 1.27)) hide)
+    )
+    (property "Mouser Part Number" "262-BMI323" (at 215.9 616.84 0)
+      (effects (font (size 1.27 1.27)) (justify left top) hide)
+    )
+    (property "Mouser Price/Stock" "https://www.mouser.co.uk/ProductDetail/Bosch-Sensortec/BMI323?qs=By6Nw2ByBD3%2FE1v0UqNQPQ%3D%3D" (at 215.9 716.84 0)
+      (effects (font (size 1.27 1.27)) (justify left top) hide)
+    )
+    (property "Manufacturer_Name" "BOSCH" (at 215.9 816.84 0)
+      (effects (font (size 1.27 1.27)) (justify left top) hide)
+    )
+    (property "Manufacturer_Part_Number" "BMI323" (at 215.9 916.84 0)
+      (effects (font (size 1.27 1.27)) (justify left top) hide)
     )
     (pin "1")
@@
       (effects (font (size 1.27 1.27)) (justify right))
     )
-    (property "Footprint" "Resistor_SMD:R_0201_0603Metric_Pad0.64x0.40mm_HandSolder" (at 186.69 144.78 0)
-      (effects (font (size 1.27 1.27)) hide)
-    )
+    (property "Footprint" "Resistor_SMD:R_0201_0603Metric" (at 186.69 144.78 0)
+      (effects (font (size 1.27 1.27)) hide)
+    )

Commit message: added missing MFN numbers
Parts:
- C25, C8, IC2, R3: sourced (none) -> y
- U3: MFN (none) -> 262-BMM350; sourced (none) -> y
Changed lines of the file:
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@@
+      (effects (font (size 1.27 1.27)) hide)
+    )
+    (property "MFN" "262-BMM350 " (at 322.58 130.81 0)
+      (effects (font (size 1.27 1.27)) hide)
+    )
+    (property "sourced" "y" (at 322.58 130.81 0)
       (effects (font (size 1.27 1.27)) hide)
     )
@@
       (effects (font (size 1.27 1.27)) hide)
     )
+    (property "sourced" "y" (at 171.45 116.84 0)
+      (effects (font (size 1.27 1.27)) hide)
+    )
     (pin "1")
     (pin "2")
@@
     (property "Manufacturer_Part_Number" "BMI323" (at 215.9 916.84 0)
       (effects (font (size 1.27 1.27)) (justify left top) hide)
+    )
+    (property "sourced" "y" (at 189.23 129.54 0)
+      (effects (font (size 1.27 1.27)) hide)
     )
     (pin "1")
@@
       (effects (font (size 1.27 1.27)) hide)
     )
+    (property "sourced" "y" (at 302.26 115.57 0)
+      (effects (font (size 1.27 1.27)) hide)
+    )
     (pin "1")
     (pin "2")
@@
       (effects (font (size 1.27 1.27)) hide)
     )
+    (property "sourced" "y" (at 287.02 115.57 0)
+      (effects (font (size 1.27 1.27)) hide)
+    )
     (pin "1")
     (pin "2")
@@
       (effects (font (size 1.27 1.27)) hide)
     )
+    (property "sourced" "y" (at 347.98 130.81 0)
+      (effects (font (size 1.27 1.27)) hide)
+    )
     (pin "1")
     (pin "2")
@@
       (effects (font (size 1.27 1.27)) hide)
     )
+    (property "sourced" "y" (at 156.21 116.84 0)
+      (effects (font (size 1.27 1.27)) hide)
+    )
     (pin "1")
     (pin "2")
@@
       (effects (font (size 1.27 1.27)) hide)
     )
+    (property "sourced" "y" (at 186.69 144.78 0)
+      (effects (font (size 1.27 1.27)) hide)
+    )

Commit message: Update to KiCad 8 + Add/Fix voltage selector for nRF
Parts:
- renumbered C25 to C40, C25 to C41, C8 to C42, C25 to C7, C25 to C8, R3 to R6
