File: display.kicad_sch (KiCad schematic)
At the start: 1 part, among them J3 AXF5D3012

Commit message: first layout iteration
Changed lines of the file:
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@@
     (stroke (width 0) (type default))
   )
-  (wire (pts (xy 140.97 36.83) (xy 140.97 63.5))
+  (wire (pts (xy 140.97 60.96) (xy 140.97 63.5))
     (stroke (width 0) (type default))
   )
@@
     )
   )
-  (symbol (lib_id "power:+1V8") (at 140.97 36.83 0) (unit 1)
-    (in_bom yes) (on_board yes) (dnp no) (fields_autoplaced)
-    (property "Reference" "#PWR028" (at 140.97 40.64 0)
+  (symbol (lib_id "power:+1V8") (at 140.97 60.96 0) (unit 1)
+    (in_bom yes) (on_board yes) (dnp no)
+    (property "Reference" "#PWR028" (at 140.97 64.77 0)
       (effects (font (size 1.27 1.27)) hide)
     )
-    (property "Value" "+1V8" (at 140.97 33.02 0)
+    (property "Value" "+1V8" (at 140.97 57.15 0)
       (effects (font (size 1.27 1.27)))
     )
-    (property "Footprint" "" (at 140.97 36.83 0)
+    (property "Footprint" "" (at 140.97 60.96 0)
       (effects (font (size 1.27 1.27)) hide)
     )
-    (property "Datasheet" "" (at 140.97 36.83 0)
+    (property "Datasheet" "" (at 140.97 60.96 0)
       (effects (font (size 1.27 1.27)) hide)
     )

Commit message: added missing MFN numbers
Parts:
- J3: sourced (none) -> y
Changed lines of the file:
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@@
+      (effects (font (size 1.27 1.27)) hide)
+    )
+    (property "sourced" "y" (at 113.03 71.12 0)
       (effects (font (size 1.27 1.27)) hide)
     )
