File: light_sensor.kicad_sch (KiCad schematic)
At the start: 3 parts, among them U2 VEML3235

Commit message: added missing MFN numbers
Parts:
- C25, U2: sourced (none) -> y
- C8: MFN 81-GRM155R60J106M05D -> 81-GRM155R60J106M05D; sourced (none) -> y
Changed lines of the file:
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@@
       (effects (font (size 1.27 1.27)) (justify left))
+    )
+    (property "sourced" "y" (at 90.17 62.23 0)
+      (effects (font (size 1.27 1.27)) hide)
     )
     (pin "1")
@@
       (effects (font (size 1.27 1.27)) hide)
     )
+    (property "sourced" "y" (at 93.98 48.26 0)
+      (effects (font (size 1.27 1.27)) hide)
+    )
     (pin "1")
     (pin "2")
@@
       (effects (font (size 1.27 1.27)) hide)
     )
-    (property "MFN" " 81-GRM155R60J106M05D " (at 78.74 48.26 0)
+    (property "MFN" "81-GRM155R60J106M05D " (at 78.74 48.26 0)
       (effects (font (size 1.27 1.27)) hide)
     )
+    (property "sourced" "y" (at 78.74 48.26 0)
+      (effects (font (size 1.27 1.27)) hide)
+    )

Commit message: Update to KiCad 8 + Add/Fix voltage selector for nRF
Parts:
- renumbered C8 to C28, C25 to C29
